File: pcb/pcbs/switchplate.kicad_pcb (KiCad board)
At the start: 2 copper layers, 152.4 x 110.9 mm, 5 parts

Commit message: kicad 7.0.6
Other:
- net class Default removed

Commit message: switchplate distances
Other:
- outline, holes or cut-outs redrawn
- net class Default added: clearance 0.2, trace_width 0.25, via_dia 0.8, via_drill 0.4
